File: Power System/power.kicad_pcb (KiCad board)
At the start: 2 copper layers, 139.7 x 100.3 mm, 34 parts, among them J1 PC104_40Pin_2.54mm, J2 Charge Cable, J3 Battery Pack, J4 IDC Header, U1 ds2781e+, U2 TPS22810DBVR

Commit message: Updated PCB & fixed schematic
Parts:
- removed C7: 1 uF, Capacitor_SMD:C_1206_3216Metric_Pad1.42x1.75mm_HandSolder
- removed U2: TPS22810DBVR, TPS22810DBVR:TPS22810DBVR
- added MOSFET1: SI3865DDV-T1-GE3, SI3865DDVT1GE3:SI3865DDV-T1-GE3, F.Cu at (54.6, 77.5)
- added R10: 2.2k, Resistor_SMD:R_1206_3216Metric_Pad1.30x1.75mm_HandSolder, F.Cu at (64.8, 80.0)
- added R11: 47k, Resistor_SMD:R_1206_3216Metric_Pad1.30x1.75mm_HandSolder, F.Cu at (45.7, 74.9)
- C1, C2: footprint Capacitor_SMD:C_1206_3216Metric_Pad1.42x1.75mm_HandSolder -> Capacitor_SMD:C_1206_3216Metric_Pad1.33x1.80mm_HandSolder
- C3: value PCV1D101MCL2GS -> 10uF; footprint PCV1D101MCL2GS:PCV1D101MCL2GS -> Capacitor_SMD:C_1206_3216Metric_Pad1.33x1.80mm_HandSolder
- C4: value CAP_PC_8X7 -> 10uF; footprint PCV1D101MCL2GS:PCV1D101MCL2GS -> Capacitor_SMD:C_1206_3216Metric_Pad1.33x1.80mm_HandSolder
- C5: value 10 uF -> 1000pF; footprint Capacitor_SMD:C_1206_3216Metric_Pad1.42x1.75mm_HandSolder -> Capacitor_SMD:C_1206_3216Metric_Pad1.33x1.80mm_HandSolder
- C6: value 10 nF -> 0.01uF; footprint Capacitor_SMD:C_1206_3216Metric_Pad1.42x1.75mm_HandSolder -> Capacitor_SMD:C_1206_3216Metric_Pad1.33x1.80mm_HandSolder
- PS1: value R-535.0PA -> R-785.0-1.0; footprint R-535:CONV_R-535.0PA -> WhitworthStandard:RECOM-R-78xx-1.0
- PS2: value R-533.3PA -> R-783.3-1.0; footprint R-533:CONV_R-533.3PA -> WhitworthStandard:RECOM-R-78xx-1.0
- R1, R2, R4, R5, R6, R7, R8, R9: footprint Resistor_SMD:R_1206_3216Metric_Pad1.42x1.75mm_HandSolder -> Resistor_SMD:R_1206_3216Metric_Pad1.30x1.75mm_HandSolder
- R3: footprint Resistor_SMD:R_2010_5025Metric_Pad1.52x2.65mm_HandSolder -> Resistor_SMD:R_2010_5025Metric_Pad1.40x2.65mm_HandSolder
- moved C4 35.6 mm to (142.2, 57.1), turned to 270 degrees
- moved C3 35.0 mm to (143.5, 92.7), turned to 90 degrees
- moved PS1 21.5 mm to (154.9, 44.5), turned to 0 degrees
- moved PS2 20.7 mm to (153.7, 111.8)
- moved C5 20.0 mm to (54.3, 85.1), turned to 180 degrees
- moved R9 5.95 mm to (55.9, 90.2)
- moved C6 1.76 mm to (62.2, 83.8)
Connections:
- C3 pad 1: +5V -> +3V3
- C4 pad 1: +3V3 -> +5V
- C5 pad 1: +BATT -> +7.4V
- C5 pad 2: GND -> Net-(C5-Pad2)
- C6 pad 1: Net-(C6-Pad1) -> +BATT
- PS1 pad 1: Net-(PS1-Pad1) -> +7.4V
- PS1 pad 2: +7.4V -> GND
- PS1 pad 3: +7.4V -> +5V
- PS2 pad 1: Net-(PS2-Pad1) -> +7.4V
- PS2 pad 2: +7.4V -> GND
- PS2 pad 3: +7.4V -> +3V3
Routing:
- net Net-(C5-Pad2): track 0.00 -> 19.4 mm, vias 0 -> 2
- net +5V: track 23.8 -> 7.62 mm
- net +3V3: track 139.9 -> 156.1 mm, vias 2 -> 3
- net +BATT: track 68.0 -> 80.4 mm, vias 0 -> 2
- net +7.4V: track 17.9 -> 28.1 mm, vias 0 -> 2
- net GND: track 429.0 -> 419.2 mm
- net Net-(C6-Pad1): track 9.08 -> 0.00 mm
- net /PWR_ENABLE: track 59.3 -> 67.7 mm, vias 0 -> 2
- net Net-(MOSFET1-Pad1): track 0.00 -> 8.10 mm
- net Net-(F1-Pad1): track 27.0 -> 25.6 mm
Other:
- board text added: "John Larkin Meg Fairborn 2021"
- board text removed: "John Larkin 2020"
