File: Power System/power.sch (KiCad schematic (older format))
At the start: 25 parts, among them J1 PC104_40Pin_2.54mm, J2 Charge Cable, J3 Battery Pack, J4 IDC Header, U1 ds2781e+, U2 TPS22810DBVR

Commit message: Update footprints and symbols for power
Parts:
- C3, C4: symbol PCV1D101MCL2GS:PCV1D101MCL2GS -> power-rescue:PCV1D101MCL2GS-PCV1D101MCL2GS
- F1: symbol LittleFuse_0157004.DRT:0157004.DRT -> power-rescue:0157004.DRT-LittleFuse_0157004.DRT
- J1: symbol WhitworthStandard:PC104_40Pin_2.54mm -> power-rescue:PC104_40Pin_2.54mm-WhitworthStandard
- U1: symbol ds2781e&plus_:ds2781e+ -> power-rescue:ds2781e+-ds2781e&plus_
Changed lines of the file:
@@
 EESchema Schematic File Version 4
-LIBS:power-cache
 EELAYER 30 0
 EELAYER END
@@
 $EndComp
 $Comp
-L WhitworthStandard:PC104_40Pin_2.54mm J1
+L power-rescue:PC104_40Pin_2.54mm-WhitworthStandard J1
 U 1 1 5DB909C2
 P 9350 1800
@@
 $EndComp
 $Comp
-L PCV1D101MCL2GS:PCV1D101MCL2GS C3
+L power-rescue:PCV1D101MCL2GS-PCV1D101MCL2GS C3
 U 1 1 5E81C7DD
 P 2850 3250
@@
 $EndComp
 $Comp
-L PCV1D101MCL2GS:PCV1D101MCL2GS C4
+L power-rescue:PCV1D101MCL2GS-PCV1D101MCL2GS C4
 U 1 1 5E825AA3
 P 2850 4500
@@
 Regulated 5 V and 3.3 V
 $Comp
-L ds2781e&plus_:ds2781e+ U1
+L power-rescue:ds2781e+-ds2781e&plus_ U1
 U 1 1 5E836296
 P 2550 1500
@@
 	1250 1550 1150 1550
 $Comp
-L LittleFuse_0157004.DRT:0157004.DRT F1
+L power-rescue:0157004.DRT-LittleFuse_0157004.DRT F1
 U 1 1 5E83C5FB
 P 1350 2300

Commit message: Added new zones on schematic diagram
Parts:
- added C?: 1000pF, symbol Device:C
- added C? (x2): 10uF, symbol Device:C
- added MOSFET?: SI3865DDV-T1-GE3, TSOP6_MO-193C_VIS, symbol SI3865DDVT1GE3:SI3865DDV-T1-GE3
- added PS?: R-785.0-1.0, CONV_R-785.0-1.0, symbol WhitworthStandard:R-785.0-1.0
- added R?: 2.2k, symbol Device:R
- added R?: 47k, symbol Device:R
- added U?: R-783.3-1.0, symbol WhitworthStandard:R-783.3-1.0
- C3, C4: symbol power-rescue:PCV1D101MCL2GS-PCV1D101MCL2GS -> power-rescue:PCV1D101MCL2GS-PCV1D101MCL2GS-power-rescue
- F1: symbol power-rescue:0157004.DRT-LittleFuse_0157004.DRT -> power-rescue:0157004.DRT-LittleFuse_0157004.DRT-power-rescue
- J1: symbol power-rescue:PC104_40Pin_2.54mm-WhitworthStandard -> power-rescue:PC104_40Pin_2.54mm-WhitworthStandard-power-rescue
- U1: symbol power-rescue:ds2781e+-ds2781e&plus_ -> power-rescue:ds2781e+-ds2781e&plus_-power-rescue
Connections:
- wire segments 84 -> 102
Other:
- note added: "Old"
- note added: "Regulated 5V and 3.3V"

Commit message: Got rid of short and changed some notation
Parts:
- added C?: 0.01uF, symbol Device:C
- gave numbers to parts that had none: 1
Changed lines of the file:
@@
 L power:GNDPWR #PWR?
 U 1 1 61008655
-P 7400 5950
-F 0 "#PWR?" H 7400 5750 50  0001 C CNN
-F 1 "GNDPWR" H 7404 5796 50  0000 C CNN
-F 2 "" H 7400 5900 50  0001 C CNN
-F 3 "" H 7400 5900 50  0001 C CNN
-	1    7400 5950
+P 7400 6250
+F 0 "#PWR?" H 7400 6050 50  0001 C CNN
+F 1 "GNDPWR" H 7404 6096 50  0000 C CNN
+F 2 "" H 7400 6200 50  0001 C CNN
+F 3 "" H 7400 6200 50  0001 C CNN
+	1    7400 6250
 	1    0    0    -1
 $EndComp
@@
 $EndComp
 Wire Notes Line
-	3950 4950 7700 4950
-Wire Notes Line
-	7700 4950 7700 6550
-Wire Notes Line
-	7700 6550 3950 6550
-Wire Notes Line
 	3950 4950 3950 6550
-Text Notes 7050 6550 0    50   ~ 0
+Text Notes 7150 6550 0    50   ~ 0
 Battery Connect
 Connection ~ 7400 5950
 $Comp
-L WhitworthStandard:R-783.3-1.0 U?
+L WhitworthStandard:R-783.3-1.0 PS?
 U 1 1 61039A89
 P 1700 6700
-F 0 "U?" H 1700 7087 60  0000 C CNN
+F 0 "PS?" H 1700 7087 60  0000 C CNN
 F 1 "R-783.3-1.0" H 1700 6981 60  0000 C CNN
 F 2 "" H 1700 6700 60  0001 C CNN
@@
 Text Notes 3250 5200 0    50   ~ 0
 Old
+$Comp
+L Device:C C?
+U 1 1 60F9FDCE
+P 7400 6100
+F 0 "C?" H 7515 6146 50  0000 L CNN
+F 1 "0.01uF" H 7515 6055 50  0000 L CNN
+F 2 "" H 7438 5950 50  0001 C CNN
+F 3 "~" H 7400 6100 50  0001 C CNN
+	1    7400 6100
+	1    0    0    -1
+$EndComp
+Wire Notes Line
+	7800 4950 7800 6550
+Wire Notes Line
+	3950 6550 7800 6550
+Wire Notes Line
+	3950 4950 7800 4950
 $EndSCHEMATC

Commit message: deleted old regulator and battery connect from schematic
Parts:
- removed C3, C4: PCV1D101MCL2GS, PCV1D101MCL2GS:PCV1D101MCL2GS, symbol power-rescue:PCV1D101MCL2GS-PCV1D101MCL2GS-power-rescue
- removed C5: 10 uF, Capacitor_SMD:C_1206_3216Metric_Pad1.42x1.75mm_HandSolder, symbol Device:C
- removed C6: 10 nF, Capacitor_SMD:C_1206_3216Metric_Pad1.42x1.75mm_HandSolder, symbol Device:C
- removed C7: 1 uF, Capacitor_SMD:C_1206_3216Metric_Pad1.42x1.75mm_HandSolder, symbol Device:C
- removed PS1: R-535.0PA, R-535:CONV_R-535.0PA, symbol R-535.0PA:R-535.0PA
- removed PS2: R-533.3PA, R-533:CONV_R-533.3PA, symbol R-533.3PA:R-533.3PA
- removed U2: TPS22810DBVR, TPS22810DBVR:TPS22810DBVR, symbol TPS22810DBVR:TPS22810DBVR
Connections:
- wire segments 102 -> 85
- no-connect marks 5 -> 1
Other:
- note removed: "Old"
- note removed: "Regulated 5 V and 3.3 V"
- moved on the sheet: C?, MOSFET?, PS?, R?

Commit message: generated a netlist
Parts:
- gave numbers to parts that had none: 9
Changed lines of the file:
@@
 Connection ~ 2650 3500
 $Comp
-L power:+5V #PWR?
+L power:+5V #PWR0124
 U 1 1 6105A92E
 P 2650 3500
-F 0 "#PWR?" H 2650 3350 50  0001 C CNN
+F 0 "#PWR0124" H 2650 3350 50  0001 C CNN
 F 1 "+5V" H 2665 3673 50  0000 C CNN
 F 2 "" H 2650 3500 50  0001 C CNN
@@
 	2250 3800 2650 3800
 $Comp
-L Device:C C?
+L Device:C C4
 U 1 1 61051914
 P 2650 3650
-F 0 "C?" H 2765 3696 50  0000 L CNN
+F 0 "C4" H 2765 3696 50  0000 L CNN
 F 1 "10uF" H 2765 3605 50  0000 L CNN
 F 2 "" H 2688 3500 50  0001 C CNN
@@
 Connection ~ 2500 4500
 $Comp
-L power:+3.3V #PWR?
+L power:+3.3V #PWR0125
 U 1 1 61050898
 P 2500 4500
-F 0 "#PWR?" H 2500 4350 50  0001 C CNN
+F 0 "#PWR0125" H 2500 4350 50  0001 C CNN
 F 1 "+3.3V" H 2515 4673 50  0000 C CNN
 F 2 "" H 2500 4500 50  0001 C CNN
@@
 	1650 4850 2500 4850
 $Comp
-L Device:C C?
+L Device:C C3
 U 1 1 61040873
 P 2500 4700
-F 0 "C?" H 2615 4746 50  0000 L CNN
+F 0 "C3" H 2615 4746 50  0000 L CNN
 F 1 "10uF" H 2615 4655 50  0000 L CNN
 F 2 "" H 2538 4550 50  0001 C CNN
@@
 $EndComp
 $Comp
-L WhitworthStandard:+7.4V #PWR?
+L WhitworthStandard:+7.4V #PWR0126
 U 1 1 6103FAC0
 P 1100 4500
-F 0 "#PWR?" H 1100 4350 50  0001 C CNN
+F 0 "#PWR0126" H 1100 4350 50  0001 C CNN
 F 1 "+7.4V" H 1115 4673 50  0000 C CNN
 F 2 "" H 1100 4500 50  0001 C CNN
@@
 $EndComp
 $Comp
-L WhitworthStandard:+7.4V #PWR?
+L WhitworthStandard:+7.4V #PWR0127
 U 1 1 6103E406
 P 1050 3600
-F 0 "#PWR?" H 1050 3450 50  0001 C CNN
+F 0 "#PWR0127" H 1050 3450 50  0001 C CNN
 F 1 "+7.4V" H 1065 3773 50  0000 C CNN
 F 2 "" H 1050 3600 50  0001 C CNN
@@
 $EndComp
 $Comp
-L power:GNDPWR #PWR?
+L power:GNDPWR #PWR0130
 U 1 1 6103D394
 P 1650 4900
-F 0 "#PWR?" H 1650 4700 50  0001 C CNN
+F 0 "#PWR0130" H 1650 4700 50  0001 C CNN
 F 1 "GNDPWR" H 1654 4746 50  0000 C CNN
 F 2 "" H 1650 4850 50  0001 C CNN
@@
 $EndComp
 $Comp
-L power:GNDPWR #PWR?
+L power:GNDPWR #PWR0131
 U 1 1 6103C4A6
 P 2250 3800
-F 0 "#PWR?" H 2250 3600 50  0001 C CNN
+F 0 "#PWR0131" H 2250 3600 50  0001 C CNN
 F 1 "GNDPWR" H 2254 3646 50  0000 C CNN
 F 2 "" H 2250 3750 50  0001 C CNN
@@
 $EndComp
 $Comp
-L WhitworthStandard:R-785.0-1.0 PS?
+L WhitworthStandard:R-785.0-1.0 PS1
 U 1 1 6103AE03
 P 1650 3700
-F 0 "PS?" H 1650 4067 50  0000 C CNN
+F 0 "PS1" H 1650 4067 50  0000 C CNN
 F 1 "R-785.0-1.0" H 1650 3976 50  0000 C CNN
 F 2 "CONV_R-785.0-1.0" H 1650 3700 50  0001 L BNN
@@
 $EndComp
 $Comp
-L WhitworthStandard:R-783.3-1.0 PS?
+L WhitworthStandard:R-783.3-1.0 PS2
 U 1 1 61039A89
 P 1650 4500
-F 0 "PS?" H 1650 4887 60  0000 C CNN
+F 0 "PS2" H 1650 4887 60  0000 C CNN
 F 1 "R-783.3-1.0" H 1650 4781 60  0000 C CNN
 F 2 "" H 1650 4500 60  0001 C CNN
@@
 $EndComp
 $Comp
-L Device:C C?
+L Device:C C5
 U 1 1 60FC8038
 P 3750 5150
-F 0 "C?" H 3865 5196 50  0000 L CNN
+F 0 "C5" H 3865 5196 50  0000 L CNN
 F 1 "1000pF" H 3865 5105 50  0000 L CNN
 F 2 "" H 3788 5000 50  0001 C CNN
@@
 	4350 5000 3750 5000
 $Comp
-L WhitworthStandard:+7.4V #PWR?
+L WhitworthStandard:+7.4V #PWR0132
 U 1 1 60FF8AB1
 P 3750 5000
-F 0 "#PWR?" H 3750 4850 50  0001 C CNN
+F 0 "#PWR0132" H 3750 4850 50  0001 C CNN
 F 1 "+7.4V" H 3765 5173 50  0000 C CNN
 F 2 "" H 3750 5000 50  0001 C CNN
@@
 	7300 4050 7300 5650
 $Comp
-L Device:C C?
+L Device:C C6
 U 1 1 60F9FDCE
 P 6900 5200
-F 0 "C?" H 7015 5246 50  0000 L CNN
+F 0 "C6" H 7015 5246 50  0000 L CNN
 F 1 "0.01uF" H 7015 5155 50  0000 L CNN
 F 2 "" H 6938 5050 50  0001 C CNN
@@
 Battery Connect
 $Comp
-L power:+BATT #PWR?
+L power:+BATT #PWR0133
 U 1 1 610093D3
 P 6900 5050
-F 0 "#PWR?" H 6900 4900 50  0001 C CNN
+F 0 "#PWR0133" H 6900 4900 50  0001 C CNN
 F 1 "+BATT" H 6915 5223 50  0000 C CNN
 F 2 "" H 6900 5050 50  0001 C CNN
@@
 	6600 5050 6900 5050
 $Comp
-L power:GNDPWR #PWR?
+L power:GNDPWR #PWR0134
 U 1 1 61008655
 P 6900 5350
-F 0 "#PWR?" H 6900 5150 50  0001 C CNN
+F 0 "#PWR0134" H 6900 5150 50  0001 C CNN
 F 1 "GNDPWR" H 6904 5196 50  0000 C CNN
 F 2 "" H 6900 5300 50  0001 C CNN
@@
 	5950 4800 5950 4750
 $Comp
-L Device:R R?
+L Device:R R11
 U 1 1 60FA2E30
 P 6600 4900
-F 0 "R?" H 6670 4946 50  0000 L CNN
+F 0 "R11" H 6670 4946 50  0000 L CNN
 F 1 "47k" V 6600 4850 50  0000 L CNN
 F 2 "" V 6530 4900 50  0001 C CNN
@@
 $EndComp
 $Comp
-L power:GNDPWR #PWR?
+L power:GNDPWR #PWR0135
 U 1 1 60FA2167
 P 4050 4400
-F 0 "#PWR?" H 4050 4200 50  0001 C CNN
+F 0 "#PWR0135" H 4050 4200 50  0001 C CNN
 F 1 "GNDPWR" H 4054 4246 50  0000 C CNN
 F 2 "" H 4050 4350 50  0001 C CNN
@@
 	4350 4400 4350 4800
 $Comp
-L Device:R R?
+L Device:R R10
 U 1 1 60F8C6EF
 P 4200 4400
-F 0 "R?" V 4100 4400 50  0000 C CNN
+F 0 "R10" V 4100 4400 50  0000 C CNN
 F 1 "2.2k" V 4200 4400 50  0000 C CNN
 F 2 "" V 4130 4400 50  0001 C CNN
@@
 	4350 4900 4350 5000
 $Comp
-L SI3865DDVT1GE3:SI3865DDV-T1-GE3 MOSFET?
+L SI3865DDVT1GE3:SI3865DDV-T1-GE3 MOSFET1
 U 1 1 60F87FD2
 P 4350 4800
-F 0 "MOSFET?" H 5150 5187 60  0000 C CNN
+F 0 "MOSFET1" H 5150 5187 60  0000 C CNN
 F 1 "SI3865DDV-T1-GE3" H 5150 5081 60  0000 C CNN
 F 2 "TSOP6_MO-193C_VIS" H 5150 5040 60  0001 C CNN

Commit message: Updated PCB & fixed schematic
Parts:
- C1, C2: footprint Capacitor_SMD:C_1206_3216Metric_Pad1.42x1.75mm_HandSolder -> Capacitor_SMD:C_1206_3216Metric_Pad1.33x1.80mm_HandSolder
- C3, C4, C5, C6: footprint (none) -> Capacitor_SMD:C_1206_3216Metric_Pad1.33x1.80mm_HandSolder
- F1: symbol power-rescue:0157004.DRT-LittleFuse_0157004.DRT-power-rescue -> power-rescue:0157004.DRT-LittleFuse_0157004.DRT-power-rescue-power-rescue
- J1: symbol power-rescue:PC104_40Pin_2.54mm-WhitworthStandard-power-rescue -> power-rescue:PC104_40Pin_2.54mm-WhitworthStandard-power-rescue-power-rescue
- MOSFET1: footprint TSOP6_MO-193C_VIS -> SI3865DDVT1GE3:SI3865DDV-T1-GE3
- PS1: footprint CONV_R-785.0-1.0 -> WhitworthStandard:RECOM-R-78xx-1.0
- PS2: footprint (none) -> WhitworthStandard:RECOM-R-78xx-1.0
- R1, R2, R4, R5, R6, R7, R8, R9: footprint Resistor_SMD:R_1206_3216Metric_Pad1.42x1.75mm_HandSolder -> Resistor_SMD:R_1206_3216Metric_Pad1.30x1.75mm_HandSolder
- R10, R11: footprint (none) -> Resistor_SMD:R_1206_3216Metric_Pad1.30x1.75mm_HandSolder
- R3: footprint Resistor_SMD:R_2010_5025Metric_Pad1.52x2.65mm_HandSolder -> Resistor_SMD:R_2010_5025Metric_Pad1.40x2.65mm_HandSolder
- U1: symbol power-rescue:ds2781e+-ds2781e&plus_-power-rescue -> power-rescue:ds2781e+-ds2781e&plus_-power-rescue-power-rescue
Connections:
- net GND: now also C3.2
Changed lines of the file:
@@
 $EndComp
 $Comp
-L power-rescue:PC104_40Pin_2.54mm-WhitworthStandard-power-rescue J1
+L power-rescue:PC104_40Pin_2.54mm-WhitworthStandard-power-rescue-power-rescue J1
 U 1 1 5DB909C2
 P 9350 1800
@@
 F 0 "R7" V 8650 3650 50  0000 C CNN
 F 1 "220" V 8550 3650 50  0000 C CNN
-F 2 "Resistor_SMD:R_1206_3216Metric_Pad1.42x1.75mm_HandSolder" V 8480 3650 50  0001 C CNN
+F 2 "Resistor_SMD:R_1206_3216Metric_Pad1.30x1.75mm_HandSolder" V 8480 3650 50  0001 C CNN
 F 3 "~" H 8550 3650 50  0001 C CNN
 	1    8550 3650
@@
 F 0 "R6" V 8250 3750 50  0000 C CNN
 F 1 "220" V 8150 3750 50  0000 C CNN
-F 2 "Resistor_SMD:R_1206_3216Metric_Pad1.42x1.75mm_HandSolder" V 8080 3750 50  0001 C CNN
+F 2 "Resistor_SMD:R_1206_3216Metric_Pad1.30x1.75mm_HandSolder" V 8080 3750 50  0001 C CNN
 F 3 "~" H 8150 3750 50  0001 C CNN
 	1    8150 3750
@@
 F 0 "R5" V 7850 3850 50  0000 C CNN
 F 1 "220" V 7750 3850 50  0000 C CNN
-F 2 "Resistor_SMD:R_1206_3216Metric_Pad1.42x1.75mm_HandSolder" V 7680 3850 50  0001 C CNN
+F 2 "Resistor_SMD:R_1206_3216Metric_Pad1.30x1.75mm_HandSolder" V 7680 3850 50  0001 C CNN
 F 3 "~" H 7750 3850 50  0001 C CNN
 	1    7750 3850
@@
 F 0 "R9" H 9820 4446 50  0000 L CNN
 F 1 "47k" V 9750 4350 50  0000 L CNN
-F 2 "Resistor_SMD:R_1206_3216Metric_Pad1.42x1.75mm_HandSolder" V 9680 4400 50  0001 C CNN
+F 2 "Resistor_SMD:R_1206_3216Metric_Pad1.30x1.75mm_HandSolder" V 9680 4400 50  0001 C CNN
 F 3 "~" H 9750 4400 50  0001 C CNN
 	1    9750 4400
@@
 F 0 "R8" V 8700 4050 50  0000 L CNN
 F 1 "47k" V 8600 4050 50  0000 L CNN
-F 2 "Resistor_SMD:R_1206_3216Metric_Pad1.42x1.75mm_HandSolder" V 8530 4100 50  0001 C CNN
+F 2 "Resistor_SMD:R_1206_3216Metric_Pad1.30x1.75mm_HandSolder" V 8530 4100 50  0001 C CNN
 F 3 "~" H 8600 4100 50  0001 C CNN
 	1    8600 4100
@@
 $EndComp
 $Comp
-L power-rescue:ds2781e+-ds2781e&plus_-power-rescue U1
+L power-rescue:ds2781e+-ds2781e&plus_-power-rescue-power-rescue U1
 U 1 1 5E836296
 P 2550 1500
@@
 F 0 "R4" H 4520 2496 50  0000 L CNN
 F 1 "4.7k" V 4450 2350 50  0000 L CNN
-F 2 "Resistor_SMD:R_1206_3216Metric_Pad1.42x1.75mm_HandSolder" V 4380 2450 50  0001 C CNN
+F 2 "Resistor_SMD:R_1206_3216Metric_Pad1.30x1.75mm_HandSolder" V 4380 2450 50  0001 C CNN
 F 3 "~" H 4450 2450 50  0001 C CNN
 	1    4450 2450
@@
 F 0 "R3" V 3550 850 50  0000 C CNN
 F 1 "RSNS" V 3650 850 50  0000 C CNN
-F 2 "Resistor_SMD:R_2010_5025Metric_Pad1.52x2.65mm_HandSolder" V 3580 850 50  0001 C CNN
+F 2 "Resistor_SMD:R_2010_5025Metric_Pad1.40x2.65mm_HandSolder" V 3580 850 50  0001 C CNN
 F 3 "~" H 3650 850 50  0001 C CNN
 	1    3650 850
@@
 	1250 1550 1150 1550
 $Comp
-L power-rescue:0157004.DRT-LittleFuse_0157004.DRT-power-rescue F1
+L power-rescue:0157004.DRT-LittleFuse_0157004.DRT-power-rescue-power-rescue F1
 U 1 1 5E83C5FB
 P 1350 2300
@@
 F 0 "C1" H 2165 1396 50  0000 L CNN
 F 1 "0.1 uF" H 2165 1305 50  0000 L CNN
-F 2 "Capacitor_SMD:C_1206_3216Metric_Pad1.42x1.75mm_HandSolder" H 2088 1200 50  0001 C CNN
+F 2 "Capacitor_SMD:C_1206_3216Metric_Pad1.33x1.80mm_HandSolder" H 2088 1200 50  0001 C CNN
 F 3 "~" H 2050 1350 50  0001 C CNN
 	1    2050 1350
@@
 F 0 "R1" V 1400 1400 50  0000 C CNN
 F 1 "1k" V 1500 1400 50  0000 C CNN
-F 2 "Resistor_SMD:R_1206_3216Metric_Pad1.42x1.75mm_HandSolder" V 1430 1400 50  0001 C CNN
+F 2 "Resistor_SMD:R_1206_3216Metric_Pad1.30x1.75mm_HandSolder" V 1430 1400 50  0001 C CNN
 F 3 "~" H 1500 1400 50  0001 C CNN
 	1    1500 1400
@@
 F 0 "R2" V 1700 1800 50  0000 C CNN
 F 1 "500" V 1600 1800 50  0000 C CNN
-F 2 "Resistor_SMD:R_1206_3216Metric_Pad1.42x1.75mm_HandSolder" V 1530 1800 50  0001 C CNN
+F 2 "Resistor_SMD:R_1206_3216Metric_Pad1.30x1.75mm_HandSolder" V 1530 1800 50  0001 C CNN
 F 3 "~" H 1600 1800 50  0001 C CNN
 	1    1600 1800
@@
 F 0 "C2" H 2415 1996 50  0000 L CNN
 F 1 "0.1 uF" H 2415 1905 50  0000 L CNN
-F 2 "Capacitor_SMD:C_1206_3216Metric_Pad1.42x1.75mm_HandSolder" H 2338 1800 50  0001 C CNN
+F 2 "Capacitor_SMD:C_1206_3216Metric_Pad1.33x1.80mm_HandSolder" H 2338 1800 50  0001 C CNN
 F 3 "~" H 2300 1950 50  0001 C CNN
 	1    2300 1950
@@
 F 0 "C4" H 2765 3696 50  0000 L CNN
 F 1 "10uF" H 2765 3605 50  0000 L CNN
-F 2 "" H 2688 3500 50  0001 C CNN
+F 2 "Capacitor_SMD:C_1206_3216Metric_Pad1.33x1.80mm_HandSolder" H 2688 3500 50  0001 C CNN
 F 3 "~" H 2650 3650 50  0001 C CNN
 	1    2650 3650
@@
 Wire Wire Line
 	2200 4500 2500 4500
-Wire Wire Line
-	1650 4850 2500 4850
 $Comp
 L Device:C C3
@@
 F 0 "C3" H 2615 4746 50  0000 L CNN
 F 1 "10uF" H 2615 4655 50  0000 L CNN
-F 2 "" H 2538 4550 50  0001 C CNN
+F 2 "Capacitor_SMD:C_1206_3216Metric_Pad1.33x1.80mm_HandSolder" H 2538 4550 50  0001 C CNN
 F 3 "~" H 2500 4700 50  0001 C CNN
 	1    2500 4700
@@
 L power:GNDPWR #PWR0130
 U 1 1 6103D394
-P 1650 4900
-F 0 "#PWR0130" H 1650 4700 50  0001 C CNN
-F 1 "GNDPWR" H 1654 4746 50  0000 C CNN
-F 2 "" H 1650 4850 50  0001 C CNN
-F 3 "" H 1650 4850 50  0001 C CNN
-	1    1650 4900
+P 1650 4950
+F 0 "#PWR0130" H 1650 4750 50  0001 C CNN
+F 1 "GNDPWR" H 1654 4796 50  0000 C CNN
+F 2 "" H 1650 4900 50  0001 C CNN
+F 3 "" H 1650 4900 50  0001 C CNN
+	1    1650 4950
 	1    0    0    -1
 $EndComp
@@
 F 0 "PS1" H 1650 4067 50  0000 C CNN
 F 1 "R-785.0-1.0" H 1650 3976 50  0000 C CNN
-F 2 "CONV_R-785.0-1.0" H 1650 3700 50  0001 L BNN
+F 2 "WhitworthStandard:RECOM-R-78xx-1.0" H 1650 3700 50  0001 L BNN
 F 3 "10.20mm" H 1650 3700 50  0001 L BNN
 F 4 "RECOM" H 1650 3700 50  0001 L BNN "Field4"
@@
 $EndComp
 $Comp
-L WhitworthStandard:R-783.3-1.0 PS2
-U 1 1 61039A89
-P 1650 4500
-F 0 "PS2" H 1650 4887 60  0000 C CNN
-F 1 "R-783.3-1.0" H 1650 4781 60  0000 C CNN
-F 2 "" H 1650 4500 60  0001 C CNN
-F 3 "" H 1650 4500 60  0001 C CNN
-	1    1650 4500
-	1    0    0    -1
-$EndComp
-$Comp
 L Device:C C5
 U 1 1 60FC8038
@@
 F 0 "C5" H 3865 5196 50  0000 L CNN
 F 1 "1000pF" H 3865 5105 50  0000 L CNN
-F 2 "" H 3788 5000 50  0001 C CNN
+F 2 "Capacitor_SMD:C_1206_3216Metric_Pad1.33x1.80mm_HandSolder" H 3788 5000 50  0001 C CNN
 F 3 "~" H 3750 5150 50  0001 C CNN
 	1    3750 5150
@@
 F 0 "C6" H 7015 5246 50  0000 L CNN
 F 1 "0.01uF" H 7015 5155 50  0000 L CNN
-F 2 "" H 6938 5050 50  0001 C CNN
+F 2 "Capacitor_SMD:C_1206_3216Metric_Pad1.33x1.80mm_HandSolder" H 6938 5050 50  0001 C CNN
 F 3 "~" H 6900 5200 50  0001 C CNN
 	1    6900 5200
@@
 F 0 "R11" H 6670 4946 50  0000 L CNN
 F 1 "47k" V 6600 4850 50  0000 L CNN
-F 2 "" V 6530 4900 50  0001 C CNN
+F 2 "Resistor_SMD:R_1206_3216Metric_Pad1.30x1.75mm_HandSolder" V 6530 4900 50  0001 C CNN
 F 3 "~" H 6600 4900 50  0001 C CNN
 	1    6600 4900
@@
 F 0 "R10" V 4100 4400 50  0000 C CNN
 F 1 "2.2k" V 4200 4400 50  0000 C CNN
-F 2 "" V 4130 4400 50  0001 C CNN
+F 2 "Resistor_SMD:R_1206_3216Metric_Pad1.30x1.75mm_HandSolder" V 4130 4400 50  0001 C CNN
 F 3 "~" H 4200 4400 50  0001 C CNN
 	1    4200 4400
@@
 F 0 "MOSFET1" H 5150 5187 60  0000 C CNN
 F 1 "SI3865DDV-T1-GE3" H 5150 5081 60  0000 C CNN
-F 2 "TSOP6_MO-193C_VIS" H 5150 5040 60  0001 C CNN
+F 2 "SI3865DDVT1GE3:SI3865DDV-T1-GE3" H 5150 5040 60  0001 C CNN
 F 3 "" H 4350 4800 60  0000 C CNN
 	1    4350 4800
 	1    0    0    -1
 $EndComp
+Wire Wire Line
+	1650 4900 1650 4950
+Wire Wire Line
+	2500 4850 2500 4900
+Wire Wire Line
+	2500 4900 1650 4900
+Connection ~ 1650 4900
+$Comp
+L WhitworthStandard:R-783.3-1.0 PS2
+U 1 1 61039A89
+P 1650 4500
+F 0 "PS2" H 1650 4887 60  0000 C CNN
+F 1 "R-783.3-1.0" H 1650 4781 60  0000 C CNN
+F 2 "WhitworthStandard:RECOM-R-78xx-1.0" H 1650 4500 60  0001 C CNN
+F 3 "" H 1650 4500 60  0001 C CNN
+	1    1650 4500
+	1    0    0    -1
+$EndComp

Commit message: Pretty sure power system fill zones are done
I don't know why it wants to commit changes to the schematic?
Parts:
- F1: symbol power-rescue:0157004.DRT-LittleFuse_0157004.DRT-power-rescue-power-rescue -> power-rescue:0157004.DRT-LittleFuse_0157004.DRT-power-rescue-power-rescue-power-rescue
- J1: symbol power-rescue:PC104_40Pin_2.54mm-WhitworthStandard-power-rescue-power-rescue -> power-rescue:PC104_40Pin_2.54mm-WhitworthStandard-power-rescue-power-rescue-power-rescue
- U1: symbol power-rescue:ds2781e+-ds2781e&plus_-power-rescue-power-rescue -> power-rescue:ds2781e+-ds2781e&plus_-power-rescue-power-rescue-power-rescue
Changed lines of the file:
@@
 $EndComp
 $Comp
-L power-rescue:PC104_40Pin_2.54mm-WhitworthStandard-power-rescue-power-rescue J1
+L power-rescue:PC104_40Pin_2.54mm-WhitworthStandard-power-rescue-power-rescue-power-rescue J1
 U 1 1 5DB909C2
 P 9350 1800
@@
 $EndComp
 $Comp
-L power-rescue:ds2781e+-ds2781e&plus_-power-rescue-power-rescue U1
+L power-rescue:ds2781e+-ds2781e&plus_-power-rescue-power-rescue-power-rescue U1
 U 1 1 5E836296
 P 2550 1500
@@
 	1250 1550 1150 1550
 $Comp
-L power-rescue:0157004.DRT-LittleFuse_0157004.DRT-power-rescue-power-rescue F1
+L power-rescue:0157004.DRT-LittleFuse_0157004.DRT-power-rescue-power-rescue-power-rescue F1
 U 1 1 5E83C5FB
 P 1350 2300

Commit message: Fill zone rework
Parts:
- F1: symbol power-rescue:0157004.DRT-LittleFuse_0157004.DRT-power-rescue-power-rescue-power-rescue -> power-rescue:0157004.DRT-LittleFuse_0157004.DRT-power-rescue-power-rescue-power-rescue-power-rescue
- J1: symbol power-rescue:PC104_40Pin_2.54mm-WhitworthStandard-power-rescue-power-rescue-power-rescue -> power-rescue:PC104_40Pin_2.54mm-WhitworthStandard-power-rescue-power-rescue-power-rescue-power-rescue
- U1: symbol power-rescue:ds2781e+-ds2781e&plus_-power-rescue-power-rescue-power-rescue -> power-rescue:ds2781e+-ds2781e&plus_-power-rescue-power-rescue-power-rescue-power-rescue
Connections:
- net INTERBOARD_0 renamed AUDIO_ALERT
- net RADIO_RX renamed USB_D+
- net RADIO_TX renamed USB_B-
Changed lines of the file:
@@
 RADIO_WAKE
 Text Label 9650 1100 0    50   ~ 0
-RADIO_RX
+USB_D+
 Text Label 9650 1000 0    50   ~ 0
-RADIO_TX
+USB_B-
 Text Label 9150 1500 2    50   ~ 0
 POD_WAKE
@@
 $EndComp
 $Comp
-L power-rescue:PC104_40Pin_2.54mm-WhitworthStandard-power-rescue-power-rescue-power-rescue J1
+L power-rescue:PC104_40Pin_2.54mm-WhitworthStandard-power-rescue-power-rescue-power-rescue-power-rescue J1
 U 1 1 5DB909C2
 P 9350 1800
@@
 INTERBOARD_2
 Text Label 9650 1900 0    50   ~ 0
-INTERBOARD_0
+AUDIO_ALERT
 Text Label 9650 1600 0    50   ~ 0
 INTERBOARD_3
@@
 $EndComp
 $Comp
-L power-rescue:ds2781e+-ds2781e&plus_-power-rescue-power-rescue-power-rescue U1
+L power-rescue:ds2781e+-ds2781e&plus_-power-rescue-power-rescue-power-rescue-power-rescue U1
 U 1 1 5E836296
 P 2550 1500
@@
 	1250 1550 1150 1550
 $Comp
-L power-rescue:0157004.DRT-LittleFuse_0157004.DRT-power-rescue-power-rescue-power-rescue F1
+L power-rescue:0157004.DRT-LittleFuse_0157004.DRT-power-rescue-power-rescue-power-rescue-power-rescue F1
 U 1 1 5E83C5FB
 P 1350 2300
