File: Power System/power.sch (KiCad schematic (older format))
At the start: 26 parts, among them J1 PC104_40Pin_2.54mm, J2 Charge Cable, J3 Battery Pack, J4 IDC Header, U1 ds2781e+

Commit message: Edited values of resistors on schematic
Parts:
- F1: symbol power-rescue:0157004.DRT-LittleFuse_0157004.DRT-power-rescue-power-rescue-power-rescue-power-rescue -> power-rescue:0157004.DRT-LittleFuse_0157004.DRT-power-rescue-power-rescue-power-rescue-power-rescue-power-rescue
- J1: symbol power-rescue:PC104_40Pin_2.54mm-WhitworthStandard-power-rescue-power-rescue-power-rescue-power-rescue -> power-rescue:PC104_40Pin_2.54mm-WhitworthStandard-power-rescue-power-rescue-power-rescue-power-rescue-power-rescue
- R2: value 500 -> 499
- R5: value 220 -> 3.4
- R6: value 220 -> 5.1
- R7: value 220 -> 66.5
- U1: symbol power-rescue:ds2781e+-ds2781e&plus_-power-rescue-power-rescue-power-rescue-power-rescue -> power-rescue:ds2781e+-ds2781e&plus_-power-rescue-power-rescue-power-rescue-power-rescue-power-rescue
Changed lines of the file:
@@
 $EndComp
 $Comp
-L power-rescue:PC104_40Pin_2.54mm-WhitworthStandard-power-rescue-power-rescue-power-rescue-power-rescue J1
+L power-rescue:PC104_40Pin_2.54mm-WhitworthStandard-power-rescue-power-rescue-power-rescue-power-rescue-power-rescue J1
 U 1 1 5DB909C2
 P 9350 1800
@@
 P 8550 3650
 F 0 "R7" V 8650 3650 50  0000 C CNN
-F 1 "220" V 8550 3650 50  0000 C CNN
+F 1 "66.5" V 8550 3650 50  0000 C CNN
 F 2 "Resistor_SMD:R_1206_3216Metric_Pad1.30x1.75mm_HandSolder" V 8480 3650 50  0001 C CNN
 F 3 "~" H 8550 3650 50  0001 C CNN
@@
 P 8150 3750
 F 0 "R6" V 8250 3750 50  0000 C CNN
-F 1 "220" V 8150 3750 50  0000 C CNN
+F 1 "5.1" V 8150 3750 50  0000 C CNN
 F 2 "Resistor_SMD:R_1206_3216Metric_Pad1.30x1.75mm_HandSolder" V 8080 3750 50  0001 C CNN
 F 3 "~" H 8150 3750 50  0001 C CNN
@@
 P 7750 3850
 F 0 "R5" V 7850 3850 50  0000 C CNN
-F 1 "220" V 7750 3850 50  0000 C CNN
+F 1 "3.4" V 7750 3850 50  0000 C CNN
 F 2 "Resistor_SMD:R_1206_3216Metric_Pad1.30x1.75mm_HandSolder" V 7680 3850 50  0001 C CNN
 F 3 "~" H 7750 3850 50  0001 C CNN
@@
 $EndComp
 $Comp
-L power-rescue:ds2781e+-ds2781e&plus_-power-rescue-power-rescue-power-rescue-power-rescue U1
+L power-rescue:ds2781e+-ds2781e&plus_-power-rescue-power-rescue-power-rescue-power-rescue-power-rescue U1
 U 1 1 5E836296
 P 2550 1500
@@
 	1250 1550 1150 1550
 $Comp
-L power-rescue:0157004.DRT-LittleFuse_0157004.DRT-power-rescue-power-rescue-power-rescue-power-rescue F1
+L power-rescue:0157004.DRT-LittleFuse_0157004.DRT-power-rescue-power-rescue-power-rescue-power-rescue-power-rescue F1
 U 1 1 5E83C5FB
 P 1350 2300
@@
 P 1600 1800
 F 0 "R2" V 1700 1800 50  0000 C CNN
-F 1 "500" V 1600 1800 50  0000 C CNN
+F 1 "499" V 1600 1800 50  0000 C CNN
 F 2 "Resistor_SMD:R_1206_3216Metric_Pad1.30x1.75mm_HandSolder" V 1530 1800 50  0001 C CNN
 F 3 "~" H 1600 1800 50  0001 C CNN

Commit message: Added DC-DC Booster to schematic
Parts:
- added C? (x2): 1uF, symbol Device:C
- added C?: 22pF, symbol Device:C
- added C?: 0.47uF, symbol Device:C
- added FB?: 2.5k Ferrite Bead, symbol Device:Ferrite_Bead
- added L?: 47uH, symbol pspice:INDUCTOR
- added R?: 10k, symbol Device:R
- added R?: 243k, symbol Device:R
- added U?: LT3461AES6-TRPBF, TSOT-23_S6_LIT, symbol LT3461AES6-TRPBF?:LT3461AES6-TRPBF
- F1: symbol power-rescue:0157004.DRT-LittleFuse_0157004.DRT-power-rescue-power-rescue-power-rescue-power-rescue-power-rescue -> power-rescue:0157004.DRT-LittleFuse_0157004.DRT-power-rescue-power-rescue-power-rescue-power-rescue-power-rescue-power-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
- J1: symbol power-rescue:PC104_40Pin_2.54mm-WhitworthStandard-power-rescue-power-rescue-power-rescue-power-rescue-power-rescue -> power-rescue:PC104_40Pin_2.54mm-WhitworthStandard-power-rescue-power-rescue-power-rescue-power-rescue-power-rescue-powe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
- MOSFET1: symbol SI3865DDVT1GE3:SI3865DDV-T1-GE3 -> power-rescue:SI3865DDV-T1-GE3-SI3865DDVT1GE3
- PS1: symbol WhitworthStandard:R-785.0-1.0 -> power-rescue:R-785.0-1.0-WhitworthStandard
- U1: symbol power-rescue:ds2781e+-ds2781e&plus_-power-rescue-power-rescue-power-rescue-power-rescue-power-rescue -> power-rescue:ds2781e+-ds2781e&plus_-power-rescue-power-rescue-power-rescue-power-rescue-power-rescue-power-rescue
Connections:
- net +5V: now also C?.1, L?.2, U?.4 (*SHDN), U?.6 (VIN)
- net GND: now also C?.2, C?.2, C?.2, R?.2, U?.2 (GND)
- new net: L?.1, U?.1 (SW)
- new net: C?.2, R?.1, R?.2, U?.3 (FB)
- new net: C?.1, C?.1, FB?.2, R?.1, U?.5 (VOUT)
- new net SIPM_Power: C?.1, FB?.1
Other:
- note added: "DC-DC Booster"
- moved on the sheet: C5, C6, MOSFET1, R10, R11
