File: controller/controller.sch (KiCad schematic (older format))
At the start: 20 parts, among them J1 PC104_40Pin_2.54mm, J2 Siren, U1 FM24W256-G, U2 ZDU0110RFX, U3 ADT7410TRZ, U4 MAX732MJA883B, U5 ProteusIII

Commit message: Add PC104 connector to Whitworth Standard symbol library
Parts:
- C3, C4, C5, C6, C7, C8: symbol controller-rescue:C-Device -> controller-rescue:C-Device-controller-rescue
- D1: symbol controller-rescue:D_Zener_ALT-Device -> controller-rescue:D_Zener_ALT-Device-controller-rescue
- J1: symbol controller-rescue:PC104_40Pin_2.54mm-WhitworthStandard-controller-rescue -> WhitworthStandard:PC104_40Pin_2.54mm-WhitworthStandard
- J2: symbol controller-rescue:Screw_Terminal_01x02-Connector -> controller-rescue:Screw_Terminal_01x02-Connector-controller-rescue
- L1: symbol controller-rescue:L-Device -> controller-rescue:L-Device-controller-rescue
- MBED1: symbol controller-rescue:LPC1768-WhitworthStandard -> controller-rescue:LPC1768-WhitworthStandard-controller-rescue
- R1, R2: symbol controller-rescue:R-Device -> controller-rescue:R-Device-controller-rescue
Changed lines of the file:
@@
 $EndDescr
 $Comp
-L controller-rescue:+BATT-power #PWR0101
+L controller-rescue:+BATT-power-controller-rescue #PWR0101
 U 1 1 5DB9296C
 P 9800 900
@@
 $EndComp
 $Comp
-L controller-rescue:PWR_FLAG-power #FLG0101
+L controller-rescue:PWR_FLAG-power-controller-rescue #FLG0101
 U 1 1 5DB92D9A
 P 9800 800
@@
 	9800 800  9800 900
 $Comp
-L controller-rescue:PWR_FLAG-power #FLG0102
+L controller-rescue:PWR_FLAG-power-controller-rescue #FLG0102
 U 1 1 5DB94156
 P 10300 800
@@
 $EndComp
 $Comp
-L controller-rescue:+7.4V-WhitworthStandard #PWR0102
+L controller-rescue:+7.4V-WhitworthStandard-controller-rescue #PWR0102
 U 1 1 5DB94A82
 P 10300 900
@@
 $EndComp
 $Comp
-L controller-rescue:PWR_FLAG-power #FLG0103
+L controller-rescue:PWR_FLAG-power-controller-rescue #FLG0103
 U 1 1 5DB951CB
 P 9850 1650
@@
 $EndComp
 $Comp
-L controller-rescue:+3.3V-power #PWR0103
+L controller-rescue:+3.3V-power-controller-rescue #PWR0103
 U 1 1 5DB958B5
 P 10300 1750
@@
 $EndComp
 $Comp
-L controller-rescue:PWR_FLAG-power #FLG0104
+L controller-rescue:PWR_FLAG-power-controller-rescue #FLG0104
 U 1 1 5DB95EE2
 P 10300 1650
@@
 $EndComp
 $Comp
-L controller-rescue:+5V-power #PWR0104
+L controller-rescue:+5V-power-controller-rescue #PWR0104
 U 1 1 5DB96D50
 P 9850 1750
@@
 $EndComp
 $Comp
-L controller-rescue:PWR_FLAG-power #FLG0105
+L controller-rescue:PWR_FLAG-power-controller-rescue #FLG0105
 U 1 1 5DB978AF
 P 9400 2500
@@
 $EndComp
 $Comp
-L controller-rescue:GND-power #PWR0105
+L controller-rescue:GND-power-controller-rescue #PWR0105
 U 1 1 5DB97F49
 P 9400 2600
@@
 DIO1
 $Comp
-L controller-rescue:+5V-power #PWR0106
+L controller-rescue:+5V-power-controller-rescue #PWR0106
 U 1 1 5DBA9AD1
 P 8400 850
@@
 $EndComp
 $Comp
-L controller-rescue:GND-power #PWR0107
+L controller-rescue:GND-power-controller-rescue #PWR0107
 U 1 1 5DBAA285
 P 7350 850
@@
 $EndComp
 $Comp
-L controller-rescue:GNDS-power #PWR0108
+L controller-rescue:GNDS-power-controller-rescue #PWR0108
 U 1 1 5DBABCBA
 P 7300 1950
@@
 $EndComp
 $Comp
-L controller-rescue:GND-power #PWR0110
+L controller-rescue:GND-power-controller-rescue #PWR0110
 U 1 1 5DBB128C
 P 7900 2750
@@
 $EndComp
 $Comp
-L controller-rescue:PC104_40Pin_2.54mm-WhitworthStandard-controller-rescue J1
+L WhitworthStandard:PC104_40Pin_2.54mm-WhitworthStandard J1
 U 1 1 5DB909C2
 P 8100 1750
@@
 $EndComp
 $Comp
-L controller-rescue:+7.4V-WhitworthStandard #PWR0112
+L controller-rescue:+7.4V-WhitworthStandard-controller-rescue #PWR0112
 U 1 1 5E1E31F7
 P 7900 2550
@@
 A3
 $Comp
-L controller-rescue:+7.4V-WhitworthStandard #PWR0114
+L controller-rescue:+7.4V-WhitworthStandard-controller-rescue #PWR0114
 U 1 1 5E1EC1FF
 P 8400 2550
@@
 $EndComp
 $Comp
-L controller-rescue:GNDPWR-power #PWR0116
+L controller-rescue:GNDPWR-power-controller-rescue #PWR0116
 U 1 1 5E1F1571
 P 9850 2650
@@
 $EndComp
 $Comp
-L controller-rescue:PWR_FLAG-power #FLG0106
+L controller-rescue:PWR_FLAG-power-controller-rescue #FLG0106
 U 1 1 5E1F21ED
 P 9850 2500
@@
 $EndComp
 $Comp
-L controller-rescue:PWR_FLAG-power #FLG0107
+L controller-rescue:PWR_FLAG-power-controller-rescue #FLG0107
 U 1 1 5E1F350A
 P 10300 2500
@@
 $EndComp
 $Comp
-L controller-rescue:GNDS-power #PWR0117
+L controller-rescue:GNDS-power-controller-rescue #PWR0117
 U 1 1 5E1F3E4B
 P 10300 2650
@@
 	10300 2500 10300 2650
 $Comp
-L controller-rescue:LPC1768-WhitworthStandard MBED1
+L controller-rescue:LPC1768-WhitworthStandard-controller-rescue MBED1
 U 1 1 5E1E1462
 P 5700 4250
@@
 $EndComp
 $Comp
-L controller-rescue:GND-power #PWR0118
+L controller-rescue:GND-power-controller-rescue #PWR0118
 U 1 1 5E1E6F45
 P 4500 3300
@@
 NoConn ~ 6450 4000
 $Comp
-L controller-rescue:GND-power #PWR0120
+L controller-rescue:GND-power-controller-rescue #PWR0120
 U 1 1 5E2103DF
 P 10200 3850
@@
 I2C_SDA
 $Comp
-L controller-rescue:+3.3V-power #PWR0121
+L controller-rescue:+3.3V-power-controller-rescue #PWR0121
 U 1 1 5E211018
 P 7850 3750
@@
 NoConn ~ 1300 5000
 $Comp
-L controller-rescue:GND-power #PWR0122
+L controller-rescue:GND-power-controller-rescue #PWR0122
 U 1 1 5E68D194
 P 750 4800
@@
 I2C_SCL
 $Comp
-L controller-rescue:+3.3V-power #PWR0123
+L controller-rescue:+3.3V-power-controller-rescue #PWR0123
 U 1 1 5E6908E7
 P 1100 4300
@@
 $EndComp
 $Comp
-L controller-rescue:R-Device R1
+L controller-rescue:R-Device-controller-rescue R1
 U 1 1 5E691908
 P 1100 4450
@@
 Connection ~ 1100 4700
 $Comp
-L controller-rescue:+3.3V-power #PWR0124
+L controller-rescue:+3.3V-power-controller-rescue #PWR0124
 U 1 1 5E698065
 P 3500 4700
@@
 $EndComp
 $Comp
-L controller-rescue:R-Device R2
+L controller-rescue:R-Device-controller-rescue R2
 U 1 1 5E698CA6
 P 3650 4850
@@
 Connection ~ 7850 3950
 $Comp
-L controller-rescue:GND-power #PWR0132
+L controller-rescue:GND-power-controller-rescue #PWR0132
 U 1 1 5E716AE3
 P 7400 3950
@@
 	7250 3100 7250 4850
 $Comp
-L controller-rescue:+7.4V-WhitworthStandard #PWR0119
+L controller-rescue:+7.4V-WhitworthStandard-controller-rescue #PWR0119
 U 1 1 5E716768
 P 4950 3400
@@
 $EndComp
 $Comp
-L controller-rescue:+3.3V-power #PWR0109
+L controller-rescue:+3.3V-power-controller-rescue #PWR0109
 U 1 1 5E718EAD
 P 8400 2750
@@
 AUDIO_ALERT
 $Comp
-L controller-rescue:C-Device C7
+L controller-rescue:C-Device-controller-rescue C7
 U 1 1 5E790961
 P 3500 5850
@@
 $EndComp
 $Comp
-L controller-rescue:C-Device C6
+L controller-rescue:C-Device-controller-rescue C6
 U 1 1 5E79140F
 P 2950 5850
@@
 $EndComp
 $Comp
-L controller-rescue:GND-power #PWR0135
+L controller-rescue:GND-power-controller-rescue #PWR0135
 U 1 1 5E793608
 P 3500 6000
@@
 $EndComp
 $Comp
-L controller-rescue:GND-power #PWR0136
+L controller-rescue:GND-power-controller-rescue #PWR0136
 U 1 1 5E793E53
 P 2950 6000
@@
 Connection ~ 3500 5700
 $Comp
-L controller-rescue:+5V-power #PWR0137
+L controller-rescue:+5V-power-controller-rescue #PWR0137
 U 1 1 5E79E424
 P 2950 5700
@@
 Connection ~ 2950 5700
 $Comp
-L controller-rescue:L-Device L1
+L controller-rescue:L-Device-controller-rescue L1
 U 1 1 5E79EA23
 P 4450 6550
@@
 $EndComp
 $Comp
-L controller-rescue:D_Zener_ALT-Device D1
+L controller-rescue:D_Zener_ALT-Device-controller-rescue D1
 U 1 1 5E79F74F
 P 4850 6700
@@
 $EndComp
 $Comp
-L controller-rescue:GND-power #PWR0138
+L controller-rescue:GND-power-controller-rescue #PWR0138
 U 1 1 5E7AD985
 P 3950 6800
@@
 Connection ~ 5200 6700
 $Comp
-L controller-rescue:GND-power #PWR0139
+L controller-rescue:GND-power-controller-rescue #PWR0139
 U 1 1 5E7BFD3D
 P 5400 7100
@@
 	3950 6300 3950 6500
 $Comp
-L controller-rescue:C-Device C8
+L controller-rescue:C-Device-controller-rescue C8
 U 1 1 5E7D2A0C
 P 4150 7100
@@
 $EndComp
 $Comp
-L controller-rescue:GND-power #PWR0140
+L controller-rescue:GND-power-controller-rescue #PWR0140
 U 1 1 5E7D36C8
 P 1550 7550
@@
 	1550 7250 1550 6800
 $Comp
-L controller-rescue:C-Device C5
+L controller-rescue:C-Device-controller-rescue C5
 U 1 1 5E7D8771
 P 1550 7400
@@
 Connection ~ 1550 7250
 $Comp
-L controller-rescue:C-Device C4
+L controller-rescue:C-Device-controller-rescue C4
 U 1 1 5E7D9B3F
 P 1200 6850
@@
 $EndComp
 $Comp
-L controller-rescue:GND-power #PWR0141
+L controller-rescue:GND-power-controller-rescue #PWR0141
 U 1 1 5E7DA215
 P 1200 7000
@@
 	1550 6700 1200 6700
 $Comp
-L controller-rescue:C-Device C3
+L controller-rescue:C-Device-controller-rescue C3
 U 1 1 5E7DEECC
 P 700 6850
@@
 $EndComp
 $Comp
-L controller-rescue:GND-power #PWR0142
+L controller-rescue:GND-power-controller-rescue #PWR0142
 U 1 1 5E7DF12D
 P 700 7000
@@
 	700  6600 700  6700
 $Comp
-L controller-rescue:Screw_Terminal_01x02-Connector J2
+L controller-rescue:Screw_Terminal_01x02-Connector-controller-rescue J2
 U 1 1 5E7E19E2
 P 5950 6200
@@
 Connection ~ 5400 6700
 $Comp
-L controller-rescue:GND-power #PWR0143
+L controller-rescue:GND-power-controller-rescue #PWR0143
 U 1 1 5E7E4AE0
 P 5750 6300
@@
 INTERBOARD_3
 $Comp
-L controller-rescue:GND-power #PWR0111
+L controller-rescue:GND-power-controller-rescue #PWR0111
 U 1 1 5E8BE9E2
 P 7300 2450
@@
 $EndComp
 $Comp
-L controller-rescue:+3.3V-power #PWR0113
+L controller-rescue:+3.3V-power-controller-rescue #PWR0113
 U 1 1 5E8BEF17
 P 8400 2650
@@
 $EndComp
 $Comp
-L controller-rescue:+3.3V-power #PWR0115
+L controller-rescue:+3.3V-power-controller-rescue #PWR0115
 U 1 1 5E8BF7B4
 P 7900 2650
