File: Satellite Comm/satellite_comm.sch (KiCad schematic (older format))
At the start: 4 parts, among them J1 PC104_40Pin_2.54mm, J2 RockBLOCK9603, U1 SAM-M8Q

Commit message: First commit: Proteus III PCB footprint
Parts:
- J1: symbol WhitworthStandard:PC104_40Pin_2.54mm -> satellite_comm-rescue:PC104_40Pin_2.54mm-WhitworthStandard
- J2: symbol Molex_533981071:53398-1071 -> satellite_comm-rescue:53398-1071-Molex_533981071
- U1: symbol SAM-M8Q:SAM-M8Q -> satellite_comm-rescue:SAM-M8Q-SAM-M8Q
- XB1: symbol WhitworthStandard:XBee -> satellite_comm-rescue:XBee-WhitworthStandard
Changed lines of the file:
@@
 EESchema Schematic File Version 4
-LIBS:satellite_comm-cache
 EELAYER 30 0
 EELAYER END
@@
 $EndDescr
 $Comp
-L power:+BATT #PWR0101
+L satellite_comm-rescue:+BATT-power #PWR0101
 U 1 1 5DB9296C
 P 9800 900
@@
 $EndComp
 $Comp
-L power:PWR_FLAG #FLG0101
+L satellite_comm-rescue:PWR_FLAG-power #FLG0101
 U 1 1 5DB92D9A
 P 9800 800
@@
 	9800 800  9800 900
 $Comp
-L power:PWR_FLAG #FLG0102
+L satellite_comm-rescue:PWR_FLAG-power #FLG0102
 U 1 1 5DB94156
 P 10300 800
@@
 $EndComp
 $Comp
-L WhitworthStandard:+7.4V #PWR0102
+L satellite_comm-rescue:+7.4V-WhitworthStandard #PWR0102
 U 1 1 5DB94A82
 P 10300 900
@@
 $EndComp
 $Comp
-L power:PWR_FLAG #FLG0103
+L satellite_comm-rescue:PWR_FLAG-power #FLG0103
 U 1 1 5DB951CB
 P 9800 1650
@@
 $EndComp
 $Comp
-L power:+3.3V #PWR0103
+L satellite_comm-rescue:+3.3V-power #PWR0103
 U 1 1 5DB958B5
 P 10300 1750
@@
 $EndComp
 $Comp
-L power:PWR_FLAG #FLG0104
+L satellite_comm-rescue:PWR_FLAG-power #FLG0104
 U 1 1 5DB95EE2
 P 10300 1650
@@
 $EndComp
 $Comp
-L power:+5V #PWR0104
+L satellite_comm-rescue:+5V-power #PWR0104
 U 1 1 5DB96D50
 P 9800 1750
@@
 $EndComp
 $Comp
-L power:PWR_FLAG #FLG0105
+L satellite_comm-rescue:PWR_FLAG-power #FLG0105
 U 1 1 5DB978AF
 P 9800 2500
@@
 $EndComp
 $Comp
-L power:GND #PWR0105
+L satellite_comm-rescue:GND-power #PWR0105
 U 1 1 5DB97F49
 P 9800 2600
@@
 POD_TX
 $Comp
-L power:+5V #PWR0106
+L satellite_comm-rescue:+5V-power #PWR0106
 U 1 1 5DBA9AD1
 P 8700 900
@@
 $EndComp
 $Comp
-L power:GND #PWR0107
+L satellite_comm-rescue:GND-power #PWR0107
 U 1 1 5DBAA285
 P 7700 900
@@
 $EndComp
 $Comp
-L power:GNDS #PWR0108
+L satellite_comm-rescue:GNDS-power #PWR0108
 U 1 1 5DBABCBA
 P 7600 2000
@@
 $EndComp
 $Comp
-L power:GND #PWR0110
+L satellite_comm-rescue:GND-power #PWR0110
 U 1 1 5DBB128C
 P 8200 2800
@@
 $EndComp
 $Comp
-L WhitworthStandard:PC104_40Pin_2.54mm J1
+L satellite_comm-rescue:PC104_40Pin_2.54mm-WhitworthStandard J1
 U 1 1 5DB909C2
 P 8400 1800
@@
 $EndComp
 $Comp
-L WhitworthStandard:+7.4V #PWR0112
+L satellite_comm-rescue:+7.4V-WhitworthStandard #PWR0112
 U 1 1 5E1E31F7
 P 8200 2600
@@
 A3
 $Comp
-L WhitworthStandard:+7.4V #PWR0114
+L satellite_comm-rescue:+7.4V-WhitworthStandard #PWR0114
 U 1 1 5E1EC1FF
 P 8700 2600
@@
 $EndComp
 $Comp
-L power:PWR_FLAG #FLG0107
+L satellite_comm-rescue:PWR_FLAG-power #FLG0107
 U 1 1 5E1F350A
 P 10300 2500
@@
 $EndComp
 $Comp
-L power:GNDS #PWR0117
+L satellite_comm-rescue:GNDS-power #PWR0117
 U 1 1 5E1F3E4B
 P 10300 2650
@@
 Interboard Connector
 $Comp
-L power:+3.3V #PWR0109
+L satellite_comm-rescue:+3.3V-power #PWR0109
 U 1 1 5E718EAD
 P 8700 2800
@@
 	7700 900  8200 900
 $Comp
-L power:GND #PWR0111
+L satellite_comm-rescue:GND-power #PWR0111
 U 1 1 5E8C3E58
 P 7600 2500
@@
 $EndComp
 $Comp
-L power:+3.3V #PWR0113
+L satellite_comm-rescue:+3.3V-power #PWR0113
 U 1 1 5E8C4729
 P 8700 2700
@@
 $EndComp
 $Comp
-L power:+3.3V #PWR0115
+L satellite_comm-rescue:+3.3V-power #PWR0115
 U 1 1 5E8C4953
 P 8200 2700
@@
 $EndComp
 $Comp
-L WhitworthStandard:XBee XB1
+L satellite_comm-rescue:XBee-WhitworthStandard XB1
 U 1 1 5E8CD4F1
 P 5900 1150
@@
 $EndComp
 $Comp
-L SAM-M8Q:SAM-M8Q U1
+L satellite_comm-rescue:SAM-M8Q-SAM-M8Q U1
 U 1 1 5E90076A
 P 1300 3350
@@
 $EndComp
 $Comp
-L Molex_533981071:53398-1071 J2
+L satellite_comm-rescue:53398-1071-Molex_533981071 J2
 U 1 1 5E9026D6
 P 8500 3850
@@
 IRIDIUM_PWR_CTRL
 $Comp
-L power:+5V #PWR0116
+L satellite_comm-rescue:+5V-power #PWR0116
 U 1 1 5E90A24E
 P 8100 4150
@@
 $EndComp
 $Comp
-L power:GND #PWR0118
+L satellite_comm-rescue:GND-power #PWR0118
 U 1 1 5E90A95A
 P 8100 4350
@@
 NoConn ~ 8100 4250
 $Comp
-L power:+3.3V #PWR?
+L satellite_comm-rescue:+3.3V-power #PWR?
 U 1 1 5E8F4873
 P 4850 1000
@@
 $EndComp
 $Comp
-L power:GND #PWR?
+L satellite_comm-rescue:GND-power #PWR?
 U 1 1 5E8F4F90
 P 4850 1900

Commit message: Deleted all caches and renamed files...
Parts:
- removed J2: RockBLOCK9603, Molex_533981071:Molex_53398-1071, symbol satellite_comm-rescue:53398-1071-Molex_533981071
- removed U1: SAM-M8Q, SAMM8Q:SAM-M8Q, symbol satellite_comm-rescue:SAM-M8Q-SAM-M8Q
- removed XB1: XBee, WhitworthStandard:xbee-standard, symbol satellite_comm-rescue:XBee-WhitworthStandard
- added C1, C2: 0.1 uF, Capacitor_SMD:C_1206_3216Metric_Pad1.42x1.75mm_HandSolder, symbol Device:C
- added C3, C4: PCV1D101MCL2GS, PCV1D101MCL2GS:PCV1D101MCL2GS, symbol PCV1D101MCL2GS:PCV1D101MCL2GS
- added C5: 10 uF, Capacitor_SMD:C_1206_3216Metric_Pad1.42x1.75mm_HandSolder, symbol Device:C
- added C6: 10 nF, Capacitor_SMD:C_1206_3216Metric_Pad1.42x1.75mm_HandSolder, symbol Device:C
- added C7: 1 uF, Capacitor_SMD:C_1206_3216Metric_Pad1.42x1.75mm_HandSolder, symbol Device:C
- added F1: 0157004.DRT, LittleFuse_0157004DRT:LittleFuse_0157004.DRT, symbol LittleFuse_0157004.DRT:0157004.DRT
- added J2: Charge Cable, TerminalBlock_4Ucon:TerminalBlock_4Ucon_1x02_P3.50mm_Horizontal, symbol Connector:Screw_Terminal_01x02
- added J3: Battery Pack, TerminalBlock_4Ucon:TerminalBlock_4Ucon_1x02_P3.50mm_Horizontal, symbol Connector:Screw_Terminal_01x02
- added J4: IDC Header, Connector_IDC:IDC-Header_2x05_P2.54mm_Vertical, symbol Connector_Generic:Conn_02x05_Counter_Clockwise
- added PS1: R-535.0PA, R-535:CONV_R-535.0PA, symbol R-535.0PA:R-535.0PA
- added PS2: R-533.3PA, R-533:CONV_R-533.3PA, symbol R-533.3PA:R-533.3PA
- added R1: 1k, Resistor_SMD:R_1206_3216Metric_Pad1.42x1.75mm_HandSolder, symbol Device:R
- added R2: 500, Resistor_SMD:R_1206_3216Metric_Pad1.42x1.75mm_HandSolder, symbol Device:R
- added R3: RSNS, Resistor_SMD:R_2010_5025Metric_Pad1.52x2.65mm_HandSolder, symbol Device:R
- added R4: 4.7k, Resistor_SMD:R_1206_3216Metric_Pad1.42x1.75mm_HandSolder, symbol Device:R
- added R5, R6, R7: 220, Resistor_SMD:R_1206_3216Metric_Pad1.42x1.75mm_HandSolder, symbol Device:R
- added R8, R9: 47k, Resistor_SMD:R_1206_3216Metric_Pad1.42x1.75mm_HandSolder, symbol Device:R
- added U1: ds2781e+, DS2781e:ds2781e&plus_, symbol ds2781e&plus_:ds2781e+
- added U2: TPS22810DBVR, TPS22810DBVR:TPS22810DBVR, symbol TPS22810DBVR:TPS22810DBVR
- J1: symbol satellite_comm-rescue:PC104_40Pin_2.54mm-WhitworthStandard -> WhitworthStandard:PC104_40Pin_2.54mm
Connections:
- net labels added: GNDPWR, PWR_ENABLE
- wire segments 9 -> 84
- no-connect marks 17 -> 5
Other:
- note added: "Battery Connect"
- note added: "Battery Monitor"
- note added: "External Interface"
- note added: "Regulated 5 V and 3.3 V"
- note removed: "Cmd Module to Pods Communication"
- note removed: "Satellite Modem Connector"
- moved on the sheet: J1

Commit message: Stared working on schematic, not all pins labeled or connected yet...
Parts:
- removed C1, C2: 0.1 uF, Capacitor_SMD:C_1206_3216Metric_Pad1.42x1.75mm_HandSolder, symbol Device:C
- removed C3, C4: PCV1D101MCL2GS, PCV1D101MCL2GS:PCV1D101MCL2GS, symbol PCV1D101MCL2GS:PCV1D101MCL2GS
- removed C5: 10 uF, Capacitor_SMD:C_1206_3216Metric_Pad1.42x1.75mm_HandSolder, symbol Device:C
- removed C6: 10 nF, Capacitor_SMD:C_1206_3216Metric_Pad1.42x1.75mm_HandSolder, symbol Device:C
- removed C7: 1 uF, Capacitor_SMD:C_1206_3216Metric_Pad1.42x1.75mm_HandSolder, symbol Device:C
- removed F1: 0157004.DRT, LittleFuse_0157004DRT:LittleFuse_0157004.DRT, symbol LittleFuse_0157004.DRT:0157004.DRT
- removed J1: PC104_40Pin_2.54mm, WhitworthStandard:PC104_40PinSocket_2.54mm, symbol WhitworthStandard:PC104_40Pin_2.54mm
- removed J2: Charge Cable, TerminalBlock_4Ucon:TerminalBlock_4Ucon_1x02_P3.50mm_Horizontal, symbol Connector:Screw_Terminal_01x02
- removed J3: Battery Pack, TerminalBlock_4Ucon:TerminalBlock_4Ucon_1x02_P3.50mm_Horizontal, symbol Connector:Screw_Terminal_01x02
- removed J4: IDC Header, Connector_IDC:IDC-Header_2x05_P2.54mm_Vertical, symbol Connector_Generic:Conn_02x05_Counter_Clockwise
- removed PS1: R-535.0PA, R-535:CONV_R-535.0PA, symbol R-535.0PA:R-535.0PA
- removed PS2: R-533.3PA, R-533:CONV_R-533.3PA, symbol R-533.3PA:R-533.3PA
- removed R1: 1k, Resistor_SMD:R_1206_3216Metric_Pad1.42x1.75mm_HandSolder, symbol Device:R
- removed R2: 500, Resistor_SMD:R_1206_3216Metric_Pad1.42x1.75mm_HandSolder, symbol Device:R
- removed R3: RSNS, Resistor_SMD:R_2010_5025Metric_Pad1.52x2.65mm_HandSolder, symbol Device:R
- removed R4: 4.7k, Resistor_SMD:R_1206_3216Metric_Pad1.42x1.75mm_HandSolder, symbol Device:R
- removed R5, R6, R7: 220, Resistor_SMD:R_1206_3216Metric_Pad1.42x1.75mm_HandSolder, symbol Device:R
- removed R8, R9: 47k, Resistor_SMD:R_1206_3216Metric_Pad1.42x1.75mm_HandSolder, symbol Device:R
- removed U1: ds2781e+, DS2781e:ds2781e&plus_, symbol ds2781e&plus_:ds2781e+
- removed U2: TPS22810DBVR, TPS22810DBVR:TPS22810DBVR, symbol TPS22810DBVR:TPS22810DBVR
- added J?: PC104_40Pin_2.54mm-WhitworthStandard, symbol WhitworthStandard:PC104_40Pin_2.54mm-WhitworthStandard
- added J?: 53398-1071, CON00318_10, symbol Molex_533981071:53398-1071
- added U?: SAM-M8Q, QFN_M-M8Q, symbol SAM-M8Q:SAM-M8Q
- added XB?: XBee, symbol WhitworthStandard:XBee
Connections:
- net labels added: IRIDIUM_CTS, IRIDIUM_RI, IRIDIUM_RTS
- net labels removed: PWR_ENABLE
- wire segments 84 -> 33
- no-connect marks 5 -> 0
Other:
- note added: "GPS Receiver"
- note added: "Iridium Modem"
- note added: "Pod Link"
- note removed: "Battery Connect"
- note removed: "Battery Monitor"
- note removed: "External Interface"
- note removed: "Regulated 5 V and 3.3 V"
